Commit message: update tiago assets

File: gibson2/data/assets/models/tiago/tiago_description/robots/tiago.urdf.xacro (robot description, xacro)
@@ -17,5 +17,8 @@
     <xacro:arg name="has_thermal_camera" default="false"/>
     <xacro:arg name="multiple" default="false"/>
+    <xacro:arg name="description_calibration_dir" default="$(find tiago_description_calibration)/urdf/calibration"/>
+    <xacro:arg name="extrinsic_calibration_dir" default="$(find tiago_description_calibration)/urdf/calibration"/>
     <xacro:arg name="namespace" default=""/>
+    <xacro:arg name="no_safety_eps" default="false"/>
     <xacro:property name="wrist_model" value="$(arg wrist_model)" />
     <xacro:property name="end_effector" value="$(arg end_effector)" />
@@ -25,4 +28,5 @@
     <xacro:property name="is_multiple" value="$(arg multiple)" />
     <xacro:property name="nsp" value="$(arg namespace)" />
+    <xacro:property name="no_safety_eps" value="$(arg no_safety_eps)" />
   <xacro:if value="$(arg arm)">
     <xacro:if value="${wrist_model not in ['wrist-2010', 'wrist-2017']}">
@@ -30,5 +34,5 @@
     </xacro:if>
   </xacro:if>
-  <xacro:if value="${end_effector not in ['false', False, 'pal-gripper', 'pal-hey5', 'schunk-wsg', 'custom']}">
+  <xacro:if value="${end_effector not in ['false', False, 'pal-gripper', 'pal-hey5', 'schunk-wsg', 'robotiq-2f-85', 'robotiq-2f-140', 'custom']}">
     <xacro:wrong_end_effector/>
   </xacro:if>
@@ -50,4 +54,5 @@
    <xacro:property name="end_effector_name"       value="${'hand' if end_effector == 'pal-hey5' else 'gripper'}"/>
    <xacro:property name="head_link_name"          value="head_2_link"/>
+   <xacro:property name="description_calibration_dir"       value="${arg description_calibration_dir}"/>
   <!-- The following included files set up definitions of parts of the robot body -->
   <!-- Base -->
@@ -59,5 +64,5 @@
     <xacro:include filename="$(find tiago_description)/urdf/arm/arm.urdf.xacro" />
     <xacro:include filename="$(find tiago_description)/urdf/end_effector/end_effector.urdf.xacro" />
-    <xacro:include filename="$(find tiago_description_calibration)/urdf/calibration/calibration_constants.urdf.xacro" />
+  <xacro:include filename="$(arg description_calibration_dir)/calibration_constants.urdf.xacro" />
   </xacro:if>
   <!-- Force Torque sensor -->
@@ -74,7 +79,10 @@
   <xacro:base_sensors name="base" laser_model="$(arg laser_model)" sonars="true" microphone="true"/>
   <xacro:tiago_torso name="torso" parent="base_link"/>
-  <xacro:head name="head" parent="torso_lift_link" camera_model="$(arg camera_model)" description_calibration_package="tiago_description_calibration"/>
+  <xacro:head name="head" parent="torso_lift_link" camera_model="$(arg camera_model)"
+	  description_calibration_dir="$(arg description_calibration_dir)"
+	  extrinsic_calibration_dir="$(arg extrinsic_calibration_dir)"
+    no_safety_eps="${no_safety_eps}"/>
   <xacro:if value="${has_arm}">
-	  <xacro:tiago_arm name="arm" parent="torso_lift_link" wrist_model="${wrist_model}" has_ft_sensor="${has_ft_sensor}" reflect="1" tiago_dual="-1" arm_1_offset="${arm_1_joint_offset}" arm_2_offset="${arm_2_joint_offset}" arm_3_offset="${arm_3_joint_offset}" arm_4_offset="${arm_4_joint_offset}" arm_5_offset="${arm_5_joint_offset}" arm_6_offset="${arm_6_joint_offset}" arm_7_offset="${arm_7_joint_offset}">
+	  <xacro:tiago_arm name="arm" parent="torso_lift_link" wrist_model="${wrist_model}" has_ft_sensor="${has_ft_sensor}" reflect="1" tiago_dual="-1" arm_1_offset="${arm_1_joint_offset}" arm_2_offset="${arm_2_joint_offset}" arm_3_offset="${arm_3_joint_offset}" arm_4_offset="${arm_4_joint_offset}" arm_5_offset="${arm_5_joint_offset}" arm_6_offset="${arm_6_joint_offset}" arm_7_offset="${arm_7_joint_offset}" no_safety_eps="${no_safety_eps}">
         <origin xyz="0.15505 0.014 -0.151" rpy="0 0 ${-90 * deg_to_rad}" />
       </xacro:tiago_arm>

File: gibson2/data/assets/models/tiago/tiago_description/urdf/arm/arm.urdf.xacro (robot description, xacro)
@@ -23,8 +23,8 @@
   <xacro:property name="arm_3_max_effort"   value="26" />
   <xacro:property name="arm_4_max_effort"   value="26" />
-  <xacro:property name="arm_eps"            value="0.07" />
   <!-- reflect: Set to 1 for a right arm, or to -1 for a left arm-->
   <!-- tiago_dual: Set to 1 for tiago dual, -1 for original tiago, changes joints 1 and 2 -->
-  <xacro:macro name="tiago_arm" params="name parent wrist_model has_ft_sensor reflect tiago_dual *origin arm_1_offset arm_2_offset arm_3_offset arm_4_offset arm_5_offset arm_6_offset arm_7_offset">
+  <xacro:macro name="tiago_arm" params="name parent wrist_model has_ft_sensor reflect tiago_dual *origin arm_1_offset arm_2_offset arm_3_offset arm_4_offset arm_5_offset arm_6_offset arm_7_offset no_safety_eps:=False">
+   <xacro:property name="arm_eps"       value="${0.00 if no_safety_eps else 0.07}"/>
     <!--************************-->
     <!--        SHOULDER        -->
@@ -110,5 +110,5 @@
       <inertial>
         <origin xyz="0.007418 -0.004361 ${reflect * -0.134194}" rpy="0.00000 0.00000 0.00000"/>
-        <mass value="2.343502"/>
+        <mass value="1.8"/>
         <inertia ixx="0.019541" ixy="${1 * -0.000105}" ixz="-0.001717"
           iyy="0.019936" iyz="${reflect * 0.000852}"
@@ -149,5 +149,5 @@
     <link name="${name}_4_link">
       <inertial>
-        <origin xyz="${reflect * -0.095658} ${reflect * 0.014666} 0.018133" rpy="0.00000 0.00000 0.00000"/>
+        <origin xyz="${reflect * -0.095658} ${reflect * 0.014666} ${reflect * 0.018133}" rpy="0.00000 0.00000 0.00000"/>
         <mass value="1.432697"/>
         <inertia ixx="0.002040" ixy="${reflect * 0.000725}" ixz="${-reflect * 0.001150}"
@@ -217,5 +217,5 @@
     <!--        WRIST           -->
     <!--************************-->
-   <xacro:wrist name="${name}" parent="${name}_4_link" reflect="${reflect}" wrist_model="${wrist_model}" has_ft_sensor="${has_ft_sensor}" arm_5_offset="${arm_5_offset}" arm_6_offset="${arm_6_offset}" arm_7_offset="${arm_7_offset}"/>
+   <xacro:wrist name="${name}" parent="${name}_4_link" reflect="${reflect}" wrist_model="${wrist_model}" has_ft_sensor="${has_ft_sensor}" arm_5_offset="${arm_5_offset}" arm_6_offset="${arm_6_offset}" arm_7_offset="${arm_7_offset}"  no_safety_eps="${no_safety_eps}"/>
     <!--***********************-->
     <!--        TOOL           -->

File: gibson2/data/assets/models/tiago/tiago_description/urdf/arm/wrist.urdf.xacro (robot description, xacro)
@@ -20,6 +20,6 @@
   <xacro:property name="wrist_2_max_effort"   value="6.6" />
   <xacro:property name="wrist_3_max_effort"   value="6.6" />
-  <xacro:property name="wrist_eps"          value="0.02" />
-  <xacro:macro name="wrist" params="name parent reflect wrist_model has_ft_sensor arm_5_offset arm_6_offset arm_7_offset">
+  <xacro:macro name="wrist" params="name parent reflect wrist_model has_ft_sensor arm_5_offset arm_6_offset arm_7_offset no_safety_eps:=False">
+   <xacro:property name="wrist_eps"       value="${0.00 if no_safety_eps else 0.02}"/>
     <!--************************-->
     <!--        WRIST           -->

File: gibson2/data/assets/models/tiago/tiago_description/urdf/end_effector/end_effector.urdf.xacro (robot description, xacro)
@@ -18,5 +18,5 @@
     - reflect: Set to 1 for a right end effector, or to -1 for a left end effector
   -->
-  <xacro:macro name="tiago_end_effector" params="name parent type reflect">
+  <xacro:macro name="tiago_end_effector" params="name parent type reflect is_dual:=false">
   <!-- PAL Gripper -->
   <xacro:if value="${type == 'pal-gripper'}">
@@ -73,6 +73,20 @@
     </link>
   </xacro:if>
+  <!-- Robotiq 2F-85 Gripper -->
+  <xacro:if value="${type == 'robotiq-2f-85'}">
+    <xacro:include filename="$(find pal_robotiq_85_description)/urdf/robotiq_85_gripper.urdf.xacro" />
+    <xacro:robotiq_85_gripper prefix="${name}_" parent="${parent}" >
+      <origin xyz="0.01 0 0" rpy="${90*deg_to_rad} ${0*deg_to_rad} ${90*deg_to_rad}"/>
+    </xacro:robotiq_85_gripper>
+  </xacro:if>
+  <!-- Robotiq 2F-140 Gripper -->
+  <xacro:if value="${type == 'robotiq-2f-140'}">
+    <xacro:include filename="$(find pal_robotiq_140_description)/urdf/robotiq_140_gripper.urdf.xacro" />
+    <xacro:robotiq_140_gripper prefix="${name}_" parent="${parent}" >
+      <origin xyz="0.01 0 0" rpy="${90*deg_to_rad} ${0*deg_to_rad} ${90*deg_to_rad}"/>
+    </xacro:robotiq_140_gripper>
+  </xacro:if>
   <!-- Custom -->
-  <xacro:if value="${type == 'custom'}">
+  <xacro:if value="${type == 'custom' and not is_dual}">
     <xacro:include filename="$(find custom_ee_description)/urdf/end-effector.urdf.xacro" />
     <xacro:end_effector parent="${parent}">
@@ -80,4 +94,19 @@
     </xacro:end_effector>
   </xacro:if>
+  <!-- Custom dual-->
+  <xacro:if value="${type == 'custom' and is_dual}">
+    <xacro:if value="${reflect == 1}"> <!-- If right -->
+    <xacro:include filename="$(find custom_dual_ee_description)/urdf/end-effector-right.urdf.xacro" />
+    <xacro:end_effector_right parent="${parent}">
+      <origin xyz="0.01 0 0" rpy="${90*deg_to_rad} ${90*deg_to_rad} ${-90*deg_to_rad}"/>
+    </xacro:end_effector_right>
+    </xacro:if>
+    <xacro:if value="${reflect == -1}"> <!-- If left -->
+    <xacro:include filename="$(find custom_dual_ee_description)/urdf/end-effector-left.urdf.xacro" />
+    <xacro:end_effector_left parent="${parent}">
+      <origin xyz="0.01 0 0" rpy="${90*deg_to_rad} ${90*deg_to_rad} ${-90*deg_to_rad}"/>
+    </xacro:end_effector_left>
+    </xacro:if>
+  </xacro:if>
   </xacro:macro>
 </robot>

File: gibson2/data/assets/models/tiago/tiago_description/urdf/head/head.urdf.xacro (robot description, xacro)
@@ -17,5 +17,4 @@
   <xacro:property name="head_damping"  value="0.5" />
   <xacro:property name="head_max_vel"  value="3.0" />
-  <xacro:property name="head_eps"      value="0.07" />
   <xacro:property name="head_1_lower_limit" value="-75"/>
   <xacro:property name="head_1_upper_limit" value="75"/>
@@ -107,15 +106,16 @@
                          k_velocity="20"
                          soft_lower_limit="${head_2_lower_limit * deg_to_rad + head_eps}"
-                         soft_upper_limit="${head_2_upper_limit * deg_to_rad}" />
+                         soft_upper_limit="${head_2_upper_limit * deg_to_rad - head_eps}" />
     </joint>
     <xacro:head_transmission name="${name}" reduction="1" offset_value="${head_2_joint_offset}"/>
   </xacro:macro>
-  <xacro:macro name="head" params="name parent camera_model description_calibration_package">
+  <xacro:macro name="head" params="name parent camera_model description_calibration_dir extrinsic_calibration_dir no_safety_eps:=False">
+    <xacro:property name="head_eps"      value="${0.00 if no_safety_eps else 0.07}" />
     <!-- includes -->
-    <xacro:include filename="$(find ${description_calibration_package})/urdf/calibration/calibration_constants.urdf.xacro" />
+    <xacro:include filename="$(arg description_calibration_dir)/calibration_constants.urdf.xacro" />
     <xacro:head_1 name="${name}_1" parent="${parent}" />
     <xacro:head_2 name="${name}_2" parent="${name}_1_link"/>
     <xacro:if value="${camera_model == 'asus-xtion'}">
-      <xacro:xtion_pro_live name="xtion" parent="${name}_2" camera_model="${camera_model}" extrinsic_package="${description_calibration_package}">
+      <xacro:xtion_pro_live name="xtion" parent="${name}_2" camera_model="${camera_model}" extrinsic_calibration_dir="${extrinsic_calibration_dir}">
         <origin xyz="${camera_position_x} ${camera_position_y} ${camera_position_z}" rpy="${camera_orientation_r} ${camera_orientation_p} ${camera_orientation_y}" />
         <!-- optical origin -->
@@ -124,5 +124,5 @@
     </xacro:if>
     <xacro:if value="${camera_model in ['orbbec-astra', 'orbbec-astra-pro']}">
-      <xacro:orbbec_astra name="xtion" parent="${name}_2" camera_model="${camera_model}" extrinsic_package="${description_calibration_package}">
+      <xacro:orbbec_astra name="xtion" parent="${name}_2" camera_model="${camera_model}" extrinsic_calibration_dir="${extrinsic_calibration_dir}">
         <origin xyz="${camera_position_x} ${camera_position_y} ${camera_position_z}" rpy="${camera_orientation_r} ${camera_orientation_p} ${camera_orientation_y}" />
         <!-- optical origin -->

File: gibson2/data/assets/models/tiago/tiago_description/urdf/sensors/orbbec_astra.urdf.xacro (robot description, xacro)
@@ -21,7 +21,7 @@
   <xacro:include filename="$(find tiago_description)/urdf/sensors/openni.gazebo.xacro" />
   <!-- Macro -->
-  <xacro:macro name="orbbec_astra" params="name parent camera_model *origin *optical_origin extrinsic_package:=tiago_description_calibration">
+  <xacro:macro name="orbbec_astra" params="name parent camera_model *origin *optical_origin extrinsic_calibration_dir">
     <!-- includes -->
-    <xacro:include filename="$(find ${extrinsic_package})/urdf/calibration/extrinsic_camera_calibration_constants.urdf.xacro" />
+    <xacro:include filename="${extrinsic_calibration_dir}/extrinsic_camera_calibration_constants.urdf.xacro" />
     <!-- frames in the center of the camera -->
     <joint name="${name}_joint" type="fixed">

File: gibson2/data/assets/models/tiago/tiago_description/urdf/sensors/xtion_pro_live.urdf.xacro (robot description, xacro)
@@ -20,7 +20,7 @@
   <xacro:include filename="$(find tiago_description)/urdf/sensors/openni.gazebo.xacro" />
   <!-- Macro -->
-  <xacro:macro name="xtion_pro_live" params="name parent camera_model *origin *optical_origin extrinsic_package:=tiago_description_calibration">
+  <xacro:macro name="xtion_pro_live" params="name parent camera_model *origin *optical_origin extrinsic_calibration_dir">
     <!-- includes -->
-    <xacro:include filename="$(find ${extrinsic_package})/urdf/calibration/extrinsic_camera_calibration_constants.urdf.xacro" />
+    <xacro:include filename="${extrinsic_calibration_dir}/extrinsic_camera_calibration_constants.urdf.xacro" />
     <!-- frames in the center of the camera -->
     <joint name="${name}_joint" type="fixed">

File: gibson2/data/assets/models/tiago/tiago_dual_description/robots/tiago_dual.urdf.xacro (robot description, xacro)
@@ -13,6 +13,6 @@
     <xacro:arg name="wrist_left_model" default="wrist-2010"/>
     <xacro:arg name="wrist_right_model" default="wrist-2010"/>
-    <xacro:arg name="end_effector_left" default="pal-hey5"/> <!-- pal-gripper, pal-hey5, schunk-wsg-->
-    <xacro:arg name="end_effector_right" default="pal-hey5"/> <!-- pal-gripper, pal-hey5, schunk-wsg-->
+    <xacro:arg name="end_effector_left" default="pal-hey5"/> <!-- pal-gripper, pal-hey5, schunk-wsg, custom-->
+    <xacro:arg name="end_effector_right" default="pal-hey5"/> <!-- pal-gripper, pal-hey5, schunk-wsg, custom-->
     <xacro:arg name="ft_sensor_left" default="schunk-ft"/> <!-- false, schunk-ft -->
     <xacro:arg name="ft_sensor_right" default="schunk-ft"/> <!-- false, schunk-ft -->
@@ -21,4 +21,6 @@
     <xacro:arg name="has_screen" default="false"/> <!-- true, false -->
     <xacro:arg name="multiple" default="false"/>
+    <xacro:arg name="description_calibration_dir" default="$(find tiago_dual_description_calibration)/urdf/calibration"/>
+    <xacro:arg name="extrinsic_calibration_dir" default="$(find tiago_dual_description_calibration)/urdf/calibration"/>
     <xacro:arg name="namespace" default=""/>
     <xacro:property name="wrist_left_model" value="$(arg wrist_left_model)" />
@@ -35,4 +37,5 @@
     <xacro:property name="is_multiple" value="$(arg multiple)" />
     <xacro:property name="nsp" value="$(arg namespace)" />
+    <xacro:property name="no_safety_eps" value="$(arg no_safety_eps)" />
   <xacro:if value="${wrist_left_model not in ['wrist-2010', 'wrist-2017']}">
     <xacro:wrong_wrist_model/>
@@ -41,8 +44,8 @@
     <xacro:wrong_wrist_model/>
   </xacro:if>
-  <xacro:if value="${end_effector_left not in ['pal-gripper', 'pal-hey5', 'schunk-wsg', 'false', False]}">
+  <xacro:if value="${end_effector_left not in ['pal-gripper', 'pal-hey5', 'schunk-wsg', 'robotiq-2f-85', 'robotiq-2f-140', 'false', False, 'custom']}">
     <xacro:wrong_end_effector_left/>
   </xacro:if>
-  <xacro:if value="${end_effector_right not in ['pal-gripper', 'pal-hey5', 'schunk-wsg', 'false', False]}">
+  <xacro:if value="${end_effector_right not in ['pal-gripper', 'pal-hey5', 'schunk-wsg', 'robotiq-2f-85', 'robotiq-2f-140', 'false', False, 'custom']}">
     <xacro:wrong_end_effector_right/>
   </xacro:if>
@@ -67,4 +70,5 @@
    <xacro:property name="end_effector_right_name"       value="${'hand_right' if end_effector_right == 'pal-hey5' else 'gripper_right'}"/>
    <xacro:property name="head_link_name"          value="head_2_link"/>
+   <xacro:property name="description_calibration_dir"       value="${arg description_calibration_dir}"/>
   <!-- The following included files set up definitions of parts of the robot body -->
   <!-- Base -->
@@ -73,5 +77,5 @@
   <xacro:include filename="$(find tiago_dual_description)/urdf/torso/torso_dual.urdf.xacro" />
   <!-- Arm -->
-  <xacro:include filename="$(find tiago_dual_description_calibration)/urdf/calibration/calibration_constants.urdf.xacro" />
+  <xacro:include filename="$(arg description_calibration_dir)/calibration_constants.urdf.xacro" />
   <xacro:include filename="$(find tiago_description)/urdf/arm/arm.urdf.xacro" />
   <!-- End Effector -->
@@ -88,8 +92,11 @@
   <xacro:base_sensors name="base" laser_model="$(arg laser_model)" sonars="true" microphone="true"/>
   <xacro:tiago_dual_torso name="torso" parent="base_link" has_screen="$(arg has_screen)"/>
-  <xacro:head name="head" parent="torso_lift_link" camera_model="$(arg camera_model)" description_calibration_package="tiago_dual_description_calibration"/>
+  <xacro:head name="head" parent="torso_lift_link" camera_model="$(arg camera_model)"
+	  description_calibration_dir="$(arg description_calibration_dir)"
+	  extrinsic_calibration_dir="$(arg extrinsic_calibration_dir)"
+    no_safety_eps="${no_safety_eps}"/>
   <!-- Left -->
   <xacro:if value="${has_arm_left}">
-	  <xacro:tiago_arm name="arm_left" parent="torso_lift_link" wrist_model="${wrist_left_model}" has_ft_sensor="${has_ft_sensor_left}" reflect="-1" tiago_dual="1" arm_1_offset="${arm_left_1_joint_offset}" arm_2_offset="${arm_left_2_joint_offset}" arm_3_offset="${arm_left_3_joint_offset}" arm_4_offset="${arm_left_4_joint_offset}" arm_5_offset="${arm_left_5_joint_offset}" arm_6_offset="${arm_left_6_joint_offset}" arm_7_offset="${arm_left_7_joint_offset}">
+	  <xacro:tiago_arm name="arm_left" parent="torso_lift_link" wrist_model="${wrist_left_model}" has_ft_sensor="${has_ft_sensor_left}" reflect="-1" tiago_dual="1" arm_1_offset="${arm_left_1_joint_offset}" arm_2_offset="${arm_left_2_joint_offset}" arm_3_offset="${arm_left_3_joint_offset}" arm_4_offset="${arm_left_4_joint_offset}" arm_5_offset="${arm_left_5_joint_offset}" arm_6_offset="${arm_left_6_joint_offset}" arm_7_offset="${arm_left_7_joint_offset}" no_safety_eps="${no_safety_eps}">
 	    <origin xyz="0.02556 0.19 -0.171" rpy="${180 * deg_to_rad} 0 ${90 * deg_to_rad}"/>
 	  </xacro:tiago_arm>
@@ -97,9 +104,9 @@
 	      <xacro:ft_sensor name="wrist_left" parent="arm_left_tool_link" />
 	  </xacro:if>
-  <xacro:tiago_end_effector name="${end_effector_left_name}" parent="${end_effector_left_link}" type="${end_effector_left}" reflect="-1"/>
+  <xacro:tiago_end_effector name="${end_effector_left_name}" parent="${end_effector_left_link}" type="${end_effector_left}" reflect="-1" is_dual="true"/>
   </xacro:if>
   <!-- Right -->
   <xacro:if value="${has_arm_right}">
-	  <xacro:tiago_arm name="arm_right" parent="torso_lift_link" wrist_model="${wrist_right_model}" has_ft_sensor="${has_ft_sensor_right}" reflect="1" tiago_dual="1" arm_1_offset="${arm_right_1_joint_offset}" arm_2_offset="${arm_right_2_joint_offset}" arm_3_offset="${arm_right_3_joint_offset}" arm_4_offset="${arm_right_4_joint_offset}" arm_5_offset="${arm_right_5_joint_offset}" arm_6_offset="${arm_right_6_joint_offset}" arm_7_offset="${arm_right_7_joint_offset}">
+	  <xacro:tiago_arm name="arm_right" parent="torso_lift_link" wrist_model="${wrist_right_model}" has_ft_sensor="${has_ft_sensor_right}" reflect="1" tiago_dual="1" arm_1_offset="${arm_right_1_joint_offset}" arm_2_offset="${arm_right_2_joint_offset}" arm_3_offset="${arm_right_3_joint_offset}" arm_4_offset="${arm_right_4_joint_offset}" arm_5_offset="${arm_right_5_joint_offset}" arm_6_offset="${arm_right_6_joint_offset}" arm_7_offset="${arm_right_7_joint_offset}"  no_safety_eps="${no_safety_eps}">
 	    <origin xyz="0.02556 -0.19 -0.171" rpy="0 0 ${-90 * deg_to_rad}"/>
 	  </xacro:tiago_arm>
@@ -107,5 +114,5 @@
 	      <xacro:ft_sensor name="wrist_right" parent="arm_right_tool_link" />
 	  </xacro:if>
-	  <xacro:tiago_end_effector name="${end_effector_right_name}" parent="${end_effector_right_link}" type="${end_effector_right}" reflect="1"/>
+	  <xacro:tiago_end_effector name="${end_effector_right_name}" parent="${end_effector_right_link}" type="${end_effector_right}" reflect="1" is_dual="true"/>
   </xacro:if>
   <!-- RGBD Laser Link -->
