Commit message: update tiago assets

File: gibson2/data/assets/models/tiago/tiago_single.urdf (robot description, URDF)
Before this commit: robot tiago, 47 links, 46 joints
Links:
- added link base_mic_back_left_link
- added link base_mic_back_right_link
- added link base_mic_front_left_link
- added link base_mic_front_right_link
- added link rgbd_laser_link, mass 0.0001
- added link wrist_ft_link, mass 0.1; collision cylinder length=0.0157 radius=0.0225; visual cylinder length=0.0157 radius=0.0225
- added link wrist_ft_tool_link, mass 0.1; collision cylinder length=0.00975 radius=0.025; visual cylinder length=0.00975 radius=0.025
- added link xtion_orbbec_aux_joint_frame, mass 0.001
- link arm_1_link: mass 2.31325 -> 1.563428; geometry collision mesh filename=package://tiago_description/meshes/arm/arm_1_collision.dae scale=1 1 1; visual mesh filename=package://tiago_description/meshes/arm/arm_1.stl scale=1 1 1
- link arm_2_link: mass 1.10224 -> 1.800397; geometry collision mesh filename=package://tiago_description/meshes/arm/arm_2_collision.dae scale=1 1 1; visual mesh filename=package://tiago_description/meshes/arm/arm_2.stl scale=1 1 1
- link arm_3_link: mass 2.42460 -> 1.8; geometry collision mesh filename=package://tiago_description/meshes/arm/arm_3_collision.dae scale=1 1 1; visual mesh filename=package://tiago_description/meshes/arm/arm_3.stl scale=1 1 1
- link arm_4_link: mass 1.45429 -> 1.432697; geometry collision mesh filename=package://tiago_description/meshes/arm/arm_4_collision.dae scale=1 1 1; visual mesh filename=package://tiago_description/meshes/arm/arm_4.stl scale=1 1 1
- link arm_5_link: mass 1.07424 -> 0.9359143689; geometry collision mesh filename=package://tiago_description/meshes/arm/arm_5_collision-wris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 scale=1 1 1; visual mesh filename=package://tiago_description/meshes/arm/arm_5-wrist-2017.stl scale=1 1 1
- link arm_6_link: mass 0.28722 -> 0.30275767222; geometry collision mesh filename=package://tiago_description/meshes/arm/arm_6_collision-wris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 scale=1 1 1; visual mesh filename=package://tiago_description/meshes/arm/arm_6-wrist-2017.stl scale=1 1 1
- link arm_7_link: mass 0.05935 -> 0.100
- link base_footprint: mass 0.001 -> None
- link base_link: geometry collision mesh filename=package://pmb2_description/meshes/base/base_collision.stl; visual mesh filename=package://pmb2_description/meshes/base/base.stl
- link head_1_link: geometry collision mesh filename=package://tiago_description/meshes/head/head_1_collision.dae scale=1 1 1; visual mesh filename=package://tiago_description/meshes/head/head_1.stl scale=1 1 1
- link head_2_link: geometry collision mesh filename=package://tiago_description/meshes/head/head_2_collision.dae scale=1 1 1; visual mesh filename=package://tiago_description/meshes/head/head_2.stl scale=1 1 1
- link ignore_caster_back_left_1_link: mass 0.101 -> 0.05144761
- link ignore_caster_back_left_2_link: mass 0.03677 -> 0.08855784; geometry collision sphere radius=0.025; visual mesh filename=package://pmb2_description/meshes/wheels/caster_2.stl
- link ignore_caster_back_right_1_link: mass 0.101 -> 0.05144761
- link ignore_caster_back_right_2_link: mass 0.03677 -> 0.08855784; geometry collision sphere radius=0.025; visual mesh filename=package://pmb2_description/meshes/wheels/caster_2.stl
- link ignore_caster_front_left_1_link: mass 0.101 -> 0.05144761
- link ignore_caster_front_left_2_link: mass 0.03677 -> 0.08855784; geometry collision sphere radius=0.025; visual mesh filename=package://pmb2_description/meshes/wheels/caster_2.stl
- link ignore_caster_front_right_1_link: mass 0.101 -> 0.05144761
- link ignore_caster_front_right_2_link: mass 0.03677 -> 0.08855784; geometry collision sphere radius=0.025; visual mesh filename=package://pmb2_description/meshes/wheels/caster_2.stl
- link torso_fixed_link: geometry collision box size=0.25 0.25 0.1; collision box size=0.4 0.25 0.04
- link torso_lift_link: geometry collision mesh filename=package://tiago_description/meshes/torso/torso_lift_collisi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 scale=1 1 1; collision mesh filename=package://tiago_description/meshes/torso/torso_lift_collisi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 scale=1 1 1
- link wheel_left_link: geometry collision sphere radius=0.0985; visual mesh filename=package://pmb2_description/meshes/wheels/wheel.stl
- link wheel_right_link: geometry collision sphere radius=0.0985; visual mesh filename=package://pmb2_description/meshes/wheels/wheel.stl
Joints:
- added joint base_mic_back_left_joint: type fixed, parent base_link, child base_mic_back_left_link, origin xyz=-0.1082 -0.0599 0.195 rpy=0 0 0
- added joint base_mic_back_right_joint: type fixed, parent base_link, child base_mic_back_right_link, origin xyz=-0.1082 -0.13789 0.195 rpy=0 0 0
- added joint base_mic_front_left_joint: type fixed, parent base_link, child base_mic_front_left_link, origin xyz=0.23182 0.03902 0.195 rpy=0 0 0
- added joint base_mic_front_right_joint: type fixed, parent base_link, child base_mic_front_right_link, origin xyz=0.23182 -0.03902 0.195 rpy=0 0 0
- added joint rgbd_laser_joint: type fixed, parent base_footprint, child rgbd_laser_link, origin xyz=-0.9 0 0 rpy=0 0 0
- added joint wrist_ft_joint: type fixed, parent arm_tool_link, child wrist_ft_link, origin xyz=0.00785 0 0 rpy=1.57079632679 0 1.57079632679
- added joint wrist_tool_joint: type fixed, parent wrist_ft_link, child wrist_ft_tool_link, origin xyz=0 0 0.012725 rpy=-1.57079632679 -1.57079632679 0
- added joint xtion_orbbec_aux_joint: type fixed, parent xtion_link, child xtion_orbbec_aux_joint_frame, origin xyz=0 0 0 rpy=0 0 0
- joint arm_1_joint: limit lower=0.0 upper=2.74889357189 effort=39.0 velocity=2.7 -> lower=0.0 upper=2.74889357189 effort=43.0 velocity=1.95
- joint arm_2_joint: limit lower=-1.57079632679 upper=1.0908307825 effort=39.0 velocity=3.66 -> lower=-1.57079632679 upper=1.0908307825 effort=43.0 velocity=1.95; origin xyz=0.125 0.0165 -0.031 rpy=1.57079632679 0.0 0.0 -> xyz=0.125 0.0195 -0.031 rpy=1.57079632679 0.0 0.0
- joint arm_3_joint: limit lower=-3.53429173529 upper=1.57079632679 effort=17.86 velocity=4.58 -> lower=-3.53429173529 upper=1.57079632679 effort=26 velocity=2.35; origin xyz=0.0895 0.0 0.0015 rpy=-1.57079632679 0.0 1.57079632679 -> xyz=0.0895 0.0 -0.0015 rpy=-1.57079632679 0.0 1.57079632679
- joint arm_4_joint: limit lower=-0.392699081699 upper=2.35619449019 effort=17.86 velocity=4.58 -> lower=-0.392699081699 upper=2.35619449019 effort=26 velocity=2.35
- joint arm_5_joint: origin xyz=-0.162 0.02 0.027 rpy=0.0 -1.57079632679 0.0 -> xyz=-0.162 0.02 0.027 rpy=1.57079632679 -1.57079632679 -1.57079632679
- joint arm_6_joint: limit lower=-1.57079632679 upper=1.57079632679 effort=6.6 velocity=1.76 -> lower=-1.41371669412 upper=1.41371669412 effort=6.6 velocity=1.76
- joint gripper_joint: parent arm_tool_link -> wrist_ft_tool_link
- joint gripper_tool_joint: parent arm_tool_link -> wrist_ft_tool_link
- joint wheel_left_joint: origin xyz=0 0.2022 0 rpy=-1.57079632679 0 0 -> xyz=0 0.2022 0.0 rpy=-1.57079632679 0 0
- joint wheel_right_joint: origin xyz=0 -0.2022 0 rpy=-1.57079632679 0 0 -> xyz=0 -0.2022 0.0 rpy=-1.57079632679 0 0
- joint xtion_depth_joint: origin xyz=0.0 0.049 0.0 rpy=0 0 0 -> xyz=0.0 0.025 0.0 rpy=0 0 0; parent xtion_link -> xtion_rgb_frame
- joint xtion_joint: origin xyz=0.0908 0.08 0 rpy=-1.57079632679 0 0 -> xyz=0.0908 0.08 0.0 rpy=-1.57079632679 0.0 0.0
- joint xtion_rgb_joint: parent xtion_link -> xtion_orbbec_aux_joint_frame
